File: psu/TR-808PSU_Rev0.1.kicad_sch (KiCad schematic)
At the start: 70 parts, among them IC1 uA7805, IC2 TA7179P, P1 1, P10 10, P11 11, P12 12, P13 13, P14 14, P15 15, P16 16, P17 17, P18 18, P19 19, P2 2, P20 20, P21 21, P22 22, P3 3, P4 4, P5 5, P6 6, P7 7, P8 8, P9 9, Q1 2SB596, Q2 2SD880, SW1A SDG5P, SW1B SDG5P, T1 N-219D (220/240V)

Commit message: Elko-Polaritaetsbalken, Sicherungshalter auf einer Hoehe
Balken am Minuspol statt Schraffur (polaritaet.py), F1-F4 auf gleicher y-Lage
(Scan-Abgleich laesst sie fest), Siebdruck-Nacharbeit nach dem KiCad-Speichern.
DRC 0 Fehler, 0 offen, Netzabstand 6,5 mm.

Co-Authored-By: Claude Sonnet 5.5 <noreply@anthropic.com>
Parts:
- C2: footprint Capacitor_THT:C_Rect_L10.3mm_W5.0mm_P7.50mm_MKS4 -> Capacitor_THT:C_Rect_L13.0mm_W4.0mm_P10.00mm_FKS3_FKP3_MKS4
- C7: footprint Capacitor_THT:C_Disc_D3.0mm_W2.0mm_P2.50mm -> Capacitor_THT:C_Disc_D5.0mm_W2.5mm_P5.00mm
- R2, R3, R4, R5, R7: footprint Resistor_THT:R_Axial_DIN0207_L6.3mm_D2.5mm_P7.62mm_Horizontal -> Resistor_THT:R_Axial_DIN0207_L6.3mm_D2.5mm_P10.16mm_Horizontal

Commit message: Schraubenloecher fuer IC1, Q1, Q2 (M3, H11-H13)
Auf der Mittelachse der Regler, 1,9 mm ueber den Seitenloechern (Bestueckungsplan).
Schaltplan mit 13 Befestigungsloechern, ERC 0, DRC 0 Fehler, Abgleich 0.

Co-Authored-By: Claude Sonnet 5.5 <noreply@anthropic.com>
Parts:
- added H11, H12, H13: M3, MountingHole:MountingHole_3.2mm_M3, symbol Mechanical:MountingHole
Connections:
- net at P9.1: now also T1.9 (9 W4)
Other:
- note added: "BEFESTIGUNG: 4 Platinenbohrungen, 6 Kuehlkoerperbohrungen (246-101A), 3 Schraubenloecher der Regler"
- note removed: "BEFESTIGUNG: 4 Platinenbohrungen und 6 Kuehlkoerperbohrungen (246-101A)"

Commit message: Regler auf einer Hoehe, Bruecken W04
IC1 auf die Hoehe von Q1/Q2 (y 47,135 mm), Bahnen ueber kurze Stuecke angebunden. D1/D2 als W04
(Platine: 2W04G; Manual W-02). Schaltplan, Stueckliste, Gerber, Ausdruck neu. ERC 0, DRC 0 Fehler, Abgleich 0.

Co-Authored-By: Claude Sonnet 5.5 <noreply@anthropic.com>
Parts:
- D1, D2: value W02 -> W04
Connections:
- net at P9.1: now also T1.9 (9 W4)
Other:
- note added: "ROLAND TR-808 - NETZTEIL PS3116-054 (220/240 V), PCB 291-405A Nachgezeichnet nach dem Service Manual (15.06.1981): Schaltbild Blatt 13, Bestueckungsplan Blatt 12, Stueckliste Blatt 10. Bauteilnummern und Anschluss- nummern 1-22 wie im Original. Brueckengleichrichter D1/D2: W04 (400 V, auf dem Geraet 2W04G); das Manual nennt W-02 (200 V), die W04 passt in dieselbe Bauform und ist ein zulaessiger E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"
- note removed: "ROLAND TR-808 - NETZTEIL PS3116-054 (220/240 V), PCB 291-405A Nachgezeichnet nach dem Service Manual (15.06.1981): Schaltbild Blatt 13, Bestueckungsplan Blatt 12, Stueckliste Blatt 10. Bauteilnummern und Anschluss- nummern 1-22 wie im Original. Variante 220/240 V (PS3116-054): C1 ECQ-U2A473MF 0,047 uF, Sicherungen CEE 250 mAT, Trafo N-219D, Netzschalter SDG5P-502. Fuer 100/117 V (PS3116-051): C1 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"
