File: psu/TR-808PSU_Rev0.2.kicad_pcb (KiCad board)
At the start: 2 copper layers, 142.9 x 119.4 mm, 70 parts, among them IC1 uA7805, IC2 TA7179P, P1 1, P10 10, P11 11, P12 12, P13 13, P14 14, P15 15, P16 16, P17 17, P18 18, P19 19, P2 2, P20 20, P21 21, P22 22, P3 3, P4 4, P5 5, P6 6, P7 7, P8 8, P9 9, Q1 2SB596, Q2 2SD880

Commit message: Rev0.2: Netzleiter SW_B weiter von SW_A weg (mind. 5,67 mm)
Dateien auf Rev0.2 umbenannt, Version auf dem Bestueckungsdruck. Sonst gleiche Schaltung, Bauteile, Masse.
Rev0.1 bleibt als Tag/Release erhalten. ERC 0, DRC 0 Fehler, Abgleich 0, Netz gegen Kleinspannung ueber 8 mm.

Co-Authored-By: Claude Sonnet 5.5 <noreply@anthropic.com>
Routing:
- net /SW_B: track 68.7 -> 72.8 mm
Other:
- board text added: "TR-808PSU Rev0.2 by DSL-man.de aka DIYSYNTH.de"
- board text removed: "TR-808PSU Rev0.1 by DSL-man.de aka DIYSYNTH.de"
Changed lines of the file:
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@@
 	(paper "A2")
 	(title_block
-		(title "TR-808PSU_Rev0.1")
+		(title "TR-808PSU_Rev0.2")
 		(rev "0.1")
 		(company "DSL-man.de")
@@
 		(fp_arc
 			(start 3.173 -1.297)
-			(mid 3.57 0)
+			(mid 3.570 0.000)
 			(end 3.173 1.297)
 			(stroke
-				(width 0.4)
+				(width 0.40)
 				(type solid)
 			)
@@
 		(fp_arc
 			(start 3.173 -1.297)
-			(mid 3.57 0)
+			(mid 3.570 0.000)
 			(end 3.173 1.297)
 			(stroke
-				(width 0.4)
+				(width 0.40)
 				(type solid)
 			)
@@
 		(fp_arc
 			(start 3.173 -1.297)
-			(mid 3.57 0)
+			(mid 3.570 0.000)
 			(end 3.173 1.297)
 			(stroke
-				(width 0.4)
+				(width 0.40)
 				(type solid)
 			)
@@
 		(layer "Edge.Cuts")
 	)
-	(gr_text "TR-808PSU Rev0.1 by DSL-man.de aka DIYSYNTH.de"
+	(gr_text "TR-808PSU Rev0.2 by DSL-man.de aka DIYSYNTH.de"
 		(at 91.29 138.845 0)
 		(layer "F.SilkS")
@@
 	)
 	(segment
-		(start 48.9528 69.4428)
-		(end 43.58 63.805)
-		(width 1)
-		(layer "B.Cu")
-		(net "/SW_B")
-	)
-	(segment
-		(start 27.795 104.79)
-		(end 45.66 104.79)
-		(width 1)
-		(layer "B.Cu")
-		(net "/SW_B")
-	)
-	(segment
-		(start 49.76 100.69)
-		(end 49.685 100.615)
-		(width 1)
-		(layer "B.Cu")
-		(net "/SW_B")
-	)
-	(segment
-		(start 45.66 104.79)
-		(end 49.76 100.69)
-		(width 1)
-		(layer "B.Cu")
-		(net "/SW_B")
-	)
-	(segment
-		(start 49.685 100.615)
-		(end 49.685 71.2105)
-		(width 1)
-		(layer "B.Cu")
-		(net "/SW_B")
-	)
-	(segment
 		(start 27.62 104.965)
 		(end 27.795 104.79)
@@
 		(net "/SW_B")
 	)
-	(arc
-		(start 49.685 71.2105)
-		(mid 49.4947 70.2538)
-		(end 48.9528 69.4428)
-		(width 1)
-		(layer "B.Cu")
-		(net "/SW_B")
-	)
 	(segment
 		(start 106.88 50.905)
@@
 		(net "/+5V")
 	)
+	(segment
+		(start 27.8000 104.7900)
+		(end 48.5000 104.7900)
+		(width 1)
+		(layer "B.Cu")
+		(net "/SW_B")
+	)
+	(segment
+		(start 48.5000 104.7900)
+		(end 52.5000 100.7900)
+		(width 1)
+		(layer "B.Cu")
+		(net "/SW_B")
+	)
+	(segment
+		(start 52.5000 100.7900)
+		(end 52.5000 72.7200)
+		(width 1)
+		(layer "B.Cu")
+		(net "/SW_B")
+	)
+	(segment
+		(start 52.5000 72.7200)
+		(end 43.5800 63.8000)
+		(width 1)
+		(layer "B.Cu")
+		(net "/SW_B")
+	)
 )
