File: psu/TR-808PSU_Rev0.3.kicad_pcb (KiCad board)
At the start: 2 copper layers, 142.9 x 119.4 mm, 70 parts, among them IC1 uA7805, IC2 TA7179P, P1 1, P10 10, P11 11, P12 12, P13 13, P14 14, P15 15, P16 16, P17 17, P18 18, P19 19, P2 2, P20 20, P21 21, P22 22, P3 3, P4 4, P5 5, P6 6, P7 7, P8 8, P9 9, Q1 2SB596, Q2 2SD880

Commit message: Rev0.3: Schraubklemmen RM5 fuer die 230-V-Primaerseite (Klemmen 1-9)
Netz, Netzschalter und Trafo-Eingang (P1-P9) als vier Phoenix-MKDS-1,5-Bloecke X1-X4 statt Loetoesen.
Schaltplan, Platine, Siebdruck mit Klemmennummern, 3D, Gerber, Ausdruck neu. ERC 0, DRC 0 Fehler, Abgleich 0.

Co-Authored-By: Claude Sonnet 5.5 <noreply@anthropic.com>
Parts:
- removed P1: 1, TR808PSU:Terminal_Pin
- removed P2: 2, TR808PSU:Terminal_Pin
- removed P3: 3, TR808PSU:Terminal_Pin
- removed P4: 4, TR808PSU:Terminal_Pin
- removed P5: 5, TR808PSU:Terminal_Pin
- removed P6: 6, TR808PSU:Terminal_Pin
- removed P7: 7, TR808PSU:Terminal_Pin
- removed P8: 8, TR808PSU:Terminal_Pin
- removed P9: 9, TR808PSU:Terminal_Pin
- added X1: 2P RM5, TerminalBlock_Phoenix:TerminalBlock_Phoenix_MKDS-1,5-2_1x02_P5.00mm_Horizontal, F.Cu at (27.6, 53.6)
- added X2: 2P RM5, TerminalBlock_Phoenix:TerminalBlock_Phoenix_MKDS-1,5-2_1x02_P5.00mm_Horizontal, F.Cu at (27.6, 72.2)
- added X3: 2P RM5, TerminalBlock_Phoenix:TerminalBlock_Phoenix_MKDS-1,5-2_1x02_P5.00mm_Horizontal, F.Cu at (27.6, 91.2)
- added X4: 3P RM5, TerminalBlock_Phoenix:TerminalBlock_Phoenix_MKDS-1,5-3_1x03_P5.00mm_Horizontal, F.Cu at (27.6, 114.8)
Routing:
- net /SW_B: track 72.8 -> 80.8 mm
- net /PRI_8: track 15.4 -> 19.3 mm
- net /MAINS_A: track 7.40 -> 5.00 mm
- net /MAINS_B: track 7.04 -> 5.00 mm
Other:
- board text added: "1"
- board text added: "2"
- board text added: "3"
- board text added: "4"
- board text added: "5"
- board text added: "6"
- board text added: "7"
- board text added: "8"
- board text added: "9"
- board text added: "TR-808PSU Rev0.3 by DSL-man.de aka DIYSYNTH.de"
- board text removed: "TR-808PSU Rev0.2 by DSL-man.de aka DIYSYNTH.de"
